File: dash_to_can/dash_to_can.kicad_pcb (KiCad board)
At the start: 2 copper layers, 127 x 127 mm, 50 parts, among them J1 AVR-ISP1, J2 Conn_02x10_Top_Bottom, Q1 2N3904, Q10 AO3401A, Q2 2N3904, Q3 2N3904, Q4 AO3401A, Q5 2N3904, Q6 AO3401A, Q7 2N3904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

Commit message: updated a bit more
Parts:
- Q10, R9: moved to B.Cu
- moved R9 60.3 mm to (96.6, 102.0), turned to 90 degrees
- moved R7 60.2 mm to (91.2, 88.0)
- moved Q10 57.8 mm to (99.3, 102.7)
- moved R2 55.2 mm to (132.8, 92.2)
- moved Q2 51.8 mm to (90.0, 91.2)
- moved C5 47.6 mm to (130.9, 80.4), turned to -90 degrees
- moved C6 46.3 mm to (132.4, 80.4), turned to -90 degrees
- moved Y1 46.3 mm to (131.5, 85.6), turned to 180 degrees
- moved R1 43.5 mm to (131.4, 82.6)
- moved R4 24.6 mm to (104.0, 79.6)
- moved Q1 15.6 mm to (103.0, 76.9)
- moved R6 1.36 mm to (136.3, 103.0)
Routing:
- net SP: track 0.00 -> 74.8 mm, vias 0 -> 1
- net CANH: track 2.70 -> 42.2 mm, vias 0 -> 1
- net Net-(U3-OSC1): track 0.00 -> 33.4 mm, vias 0 -> 6
- net Net-(U3-OSC2): track 0.00 -> 27.0 mm, vias 0 -> 4
- net Net-(U1-PD4): track 0.00 -> 21.6 mm, vias 0 -> 4
- net Net-(U1-PD3): track 0.00 -> 17.7 mm, vias 0 -> 4
- net Net-(Q10-G): track 0.00 -> 15.6 mm
- net TURN L: track 0.00 -> 14.1 mm, vias 0 -> 3
- net IMMOBI IND: track 0.00 -> 11.1 mm, vias 0 -> 1
- net +12V: track 88.3 -> 95.0 mm
- net PD4: track 0.00 -> 3.32 mm
- net Net-(U3-~{RESET}): track 0.00 -> 2.83 mm
- net SP_OUT: track 0.00 -> 2.73 mm
- net Neutral: track 14.6 -> 17.0 mm
- net GND: track 69.6 -> 71.2 mm
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
Commit message: updated even more 3.0
Routing:
- removed copper zone on B.Cu, net (none)
- removed copper zone on F.Cu, net (none)
Other:
- board size 127 x 127 mm -> 100 x 100 mm
Changed lines of the file:
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@@
 	)
 	(gr_rect
-		(start 68.5 27)
-		(end 195.5 154)
-		(stroke
-			(width 0.2)
-			(type solid)
-		)
-		(fill no)
-		(layer "Edge.Cuts")
-	)
-	(gr_rect
-		(start 88.1 58.2)
-		(end 139 109)
+		(start 74.07 27.95)
+		(end 174.07 127.95)
 		(stroke
 			(width 0.05)
@@
 		(net 75)
 	)
-	(zone
-		(net 0)
-		(net_name "")
-		(layers "F.Cu" "B.Cu")
-		(hatch edge 0.5)
-		(connect_pads
-			(clearance 0.5)
-		)
-		(min_thickness 0.25)
-		(filled_areas_thickness no)
-		(fill yes
-			(thermal_gap 0.5)
-			(thermal_bridge_width 0.5)
-			(island_removal_mode 1)
-			(island_area_min 9.999999)
-		)
-		(polygon
-			(pts
-				(xy 138.98 58.22) (xy 138.98 108.98) (xy 88.12 108.98) (xy 88.12 58.22)
-			)
-		)
-	)
 	(embedded_fonts no)
