File: dash_to_can/dash_to_can.kicad_pcb (KiCad board)
At the start: 2 copper layers, 61.1 x 74.4 mm, 64 parts, among them J1 AVR-ISP1, J2 Conn_02x10_Top_Bottom, Q1 2N3904, Q10 AO3401A, Q2 2N3904, Q3 2N3904, Q4 AO3401A, Q5 2N3904, Q6 AO3401A, Q7 2N3904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

Commit message: Few Extra Updates
Parts:
- moved R5 0.90 mm to (93.5, 58.8), turned to 90 degrees
- moved H1 0.75 mm to (92.8, 45.0)
- moved H4 0.75 mm to (92.8, 111.0)
- moved R13 0.75 mm to (115.2, 46.5)
- moved R16 0.75 mm to (123.8, 46.5)
- moved Q1 0.67 mm to (102.3, 55.9)
- moved H2 0.50 mm to (143.8, 45.0)
- moved H3 0.50 mm to (143.8, 111.0)
- moved R4 0.42 mm to (105.8, 55.9)
Routing:
- net TACHO DRIVER: track 38.3 -> 36.5 mm
- net Net-(Q9-B): track 5.95 -> 4.70 mm
- net Net-(Q3-B): track 4.50 -> 5.35 mm
- net Net-(Q7-B): track 4.77 -> 4.02 mm
- net TURN L: track 59.6 -> 59.0 mm
- net SP: track 34.0 -> 33.4 mm
- net Net-(Q1-B): track 3.80 -> 4.37 mm
- net Net-(Q4-G): track 14.0 -> 14.5 mm
- net Net-(Q10-G): track 14.2 -> 14.7 mm
- net GND: vias 117 -> 118
Other:
- board size 61.1 x 74.4 mm -> 60.8 x 74.4 mm
