File: dash_to_can/dash_to_can.kicad_sch (KiCad schematic)
At the start: 64 parts, among them J1 AVR-ISP1, J2 Conn_02x10_Top_Bottom, Q1 2N3904, Q10 AO3401A, Q2 2N3904, Q3 2N3904, Q4 AO3401A, Q5 2N3904, Q6 AO3401A, Q7 2N3904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

Commit message: FIRST DRAFT
Connections:
- net CS1 renamed R DRIVER
- net IGN: no longer names the net of J2.2 (Pin_2)
- net PB1 renamed TACHO DRIVER
- net PC1 renamed HI BEAM DRIVER
- net PC5 renamed ILLUM DRIVER
- net PD4 renamed L DRIVER
- no-connect marks 20 -> 21
Other:
- moved on the sheet: C1, C11, R11, R13, R16, R18, R19, R20, R4, R5, R7, U1
