File: dash_to_can/dash_to_can.kicad_sch (KiCad schematic)
At the start: 64 parts, among them J1 AVR-ISP1, J2 Conn_02x10_Top_Bottom, Q1 2N3904, Q10 AO3401A, Q2 2N3904, Q3 2N3904, Q4 AO3401A, Q5 2N3904, Q6 AO3401A, Q7 2N3904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

Commit message: Few Extra Updates
Parts:
- F1: value 12V 3A -> 12V 1A
Changed lines of the file:
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@@
 			)
 		)
-		(property "Value" "12V 3A"
+		(property "Value" "12V 1A"
 			(at 166.37 39.3699 0)
 			(effects
